File: Aphid-HW.kicad_pcb (KiCad board)
At the start: 4 copper layers, 60 x 40 mm, 62 parts, among them J1 USB4105-GF-A-060, J2 3020-10-0100-00, M1 Mount_M3, M2 Mount_M3, M3 Mount_M3, M4 Mount_M3, Q1 DMG1012UW-7, Q2 DMG1012UW-7, U1 USBLC6-2SC6, U2 MCP1755T-3302E/OT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

Commit message: Rework logic gates
Rename to aphid
Other:
- board text added: "Aphid v1.1 Feb 26"
- board text removed: "X-Link v1.0 Feb 26"
Changed lines of the file:
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@@
 		(layer "Edge.Cuts")
 	)
-	(gr_text "X-Link\nv1.0\nFeb 26"
+	(gr_text "Aphid\nv1.1\nFeb 26"
 		(at 73.8 88.7 0)
 		(layer "F.SilkS")

Commit message: Update PCB layout
Parts:
- removed the C19 at (92.2, 68.0)
- removed the DS1 at (98.5, 85.1)
- added C22: 100n, C_Capacitor:C_0603, F.Cu at (97.0, 72.8)
- added DS2: 150060VS55040, DS_LED:DS_0603, F.Cu at (98.5, 85.2)
- added U11: 74AHC1G14SE-7, U_IC:SC70-5, F.Cu at (92.5, 63.2)
- added U6: 74LVC1T45DW-7, U_IC:SC70-6, F.Cu at (94.5, 68.7)
- added U7: 74LVC1T45DW-7, U_IC:SC70-6, F.Cu at (94.5, 71.5)
- added U8: 74LVC1T45DW-7, U_IC:SC70-6, F.Cu at (94.5, 74.3)
- added U9: 74LVC1T45DW-7, U_IC:SC70-6, F.Cu at (94.5, 77.1)
- R12: value 1K -> 470R
- R9: value 470R -> 1K
- U5: value FXLA108BQX -> 74AHC1G14SE-7; footprint U_IC:WQFN20_05_4.5x2.5 -> U_IC:SC70-5
- moved R9 20.9 mm to (75.5, 78.8), turned to -90 degrees
- moved U5 20.8 mm to (84.6, 53.2), turned to 180 degrees
- moved R12 11.9 mm to (95.4, 85.2)
- moved C21 5.03 mm to (91.9, 72.7)
- moved R8 2.64 mm to (87.0, 53.2), turned to -90 degrees
- moved Q1 2.39 mm to (95.8, 59.9)
- moved R13 2.39 mm to (93.5, 59.9)
- moved Q2 2.29 mm to (95.8, 63.2)
- moved R14 1.14 mm to (90.2, 63.2)
- renumbered C20 to C19, C22 to C20, DS2 to DS1, U6 to U10
Connections:
- C21 pad 1: /Target/TARGET_VCC -> +3V3
- Q2 pad 1: /FTDI/RTS -> Net-(Q2-G)
- R12 pad 1: Net-(U5-B6) -> /Target/TARGET_VCC
- R12 pad 2: /Target/TARGET_SWDIO -> Net-(DS2-A)
- R14 pad 1: /FTDI/RTS -> +3V3
- R14 pad 2: GND -> /FTDI/RTS
- R8 pad 1: /FTDI/DTR -> +3V3
- R8 pad 2: GND -> /FTDI/DTR
- R9 pad 1: /Target/TARGET_VCC -> /FTDI/TDI
- R9 pad 2: Net-(DS1-A) (its old number) -> /FTDI/TDO
- U10 pad 4: /FTDI/DTR -> Net-(U10-EN)
- U4 pad 26: unconnected-(U4-ACBUS0-Pad26) -> /FTDI/SWD_OEN
- U5 pad 1: +3V3 -> unconnected-(U5-NC-Pad1)
- U5 pad 2: /FTDI/RXD -> /FTDI/DTR
- U5 pad 3: /FTDI/TXD -> GND
- U5 pad 4: unconnected-(U5-A2-Pad4) -> Net-(U10-EN)
- U5 pad 5: unconnected-(U5-A3-Pad5) -> +3V3
Routing:
- net /FTDI/TDI: track 24.1 -> 1.75 mm, vias 2 -> 0
- net +3V3: track 31.9 -> 52.5 mm, vias 13 -> 22
- net /FTDI/SWD_OEN: track 0.00 -> 19.5 mm, vias 0 -> 2
- net /Target/TARGET_VCC: track 32.5 -> 38.4 mm
- net /FTDI/SRST: track 28.3 -> 32.8 mm
- net Net-(U10-EN): track 0.00 -> 3.96 mm
- net GND: track 30.0 -> 33.4 mm, vias 179 -> 140
- net /Target/TARGET_RXD: track 15.5 -> 12.7 mm
- net Net-(U5-B6): track 2.78 -> 0.00 mm
- net /FTDI/DTR: track 19.2 -> 21.5 mm, vias 0 -> 2
- net /Target/TARGET_SWDIO: track 11.7 -> 9.44 mm
- net /FTDI/RXD: track 8.25 -> 10.4 mm
- net /Target/TARGET_DETECT: track 10.8 -> 8.76 mm, vias 0 -> 1
- net /Target/TARGET_NRST: track 11.0 -> 9.06 mm
- net Net-(Q2-G): track 0.00 -> 1.89 mm
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