File: Aphid-HW.kicad_sch (KiCad schematic)
At the start: 8 parts, among them M1 Mount_M3, M2 Mount_M3, M3 Mount_M3, M4 Mount_M3

Commit message: Rework logic gates
Rename to aphid
Other:
- sheet FTDI ports: added SWD_OEN; removed none
- sheet Target ports: added SWD_OEN; removed none
- title: X-Link -> Aphid
Changed lines of the file:
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@@
 	(paper "A4")
 	(title_block
-		(title "X-Link")
-		(date "2026-02-28")
-		(rev "v1.0")
+		(title "Aphid")
+		(date "2026-03-21")
+		(rev "v1.1")
 		(company "TL Embedded")
 	)
@@
 	(wire
 		(pts
+			(xy 127 73.66) (xy 152.4 73.66)
+		)
+		(stroke
+			(width 0)
+			(type default)
+		)
+	)
+	(wire
+		(pts
 			(xy 127 71.12) (xy 152.4 71.12)
 		)
@@
 	(wire
 		(pts
+			(xy 127 58.42) (xy 152.4 58.42)
+		)
+		(stroke
+			(width 0)
+			(type default)
+		)
+	)
+	(wire
+		(pts
+			(xy 127 76.2) (xy 152.4 76.2)
+		)
+		(stroke
+			(width 0)
+			(type default)
+		)
+	)
+	(wire
+		(pts
+			(xy 76.2 57.15) (xy 101.6 57.15)
+		)
+		(stroke
+			(width 0)
+			(type default)
+		)
+	)
+	(wire
+		(pts
+			(xy 76.2 54.61) (xy 101.6 54.61)
+		)
+		(stroke
+			(width 0)
+			(type default)
+		)
+	)
+	(wire
+		(pts
+			(xy 127 63.5) (xy 152.4 63.5)
+		)
+		(stroke
+			(width 0)
+			(type default)
+		)
+	)
+	(wire
+		(pts
+			(xy 127 55.88) (xy 152.4 55.88)
+		)
+		(stroke
+			(width 0)
+			(type default)
+		)
+	)
+	(wire
+		(pts
 			(xy 127 68.58) (xy 152.4 68.58)
-		)
-		(stroke
-			(width 0)
-			(type default)
-		)
-	)
-	(wire
-		(pts
-			(xy 127 58.42) (xy 152.4 58.42)
-		)
-		(stroke
-			(width 0)
-			(type default)
-		)
-	)
-	(wire
-		(pts
-			(xy 127 73.66) (xy 152.4 73.66)
-		)
-		(stroke
-			(width 0)
-			(type default)
-		)
-	)
-	(wire
-		(pts
-			(xy 76.2 57.15) (xy 101.6 57.15)
-		)
-		(stroke
-			(width 0)
-			(type default)
-		)
-	)
-	(wire
-		(pts
-			(xy 76.2 54.61) (xy 101.6 54.61)
-		)
-		(stroke
-			(width 0)
-			(type default)
-		)
-	)
-	(wire
-		(pts
-			(xy 127 55.88) (xy 152.4 55.88)
-		)
-		(stroke
-			(width 0)
-			(type default)
-		)
-	)
-	(wire
-		(pts
-			(xy 127 66.04) (xy 152.4 66.04)
 		)
 		(stroke
@@
 	(sheet
 		(at 152.4 50.8)
-		(size 25.4 25.4)
+		(size 25.4 27.94)
 		(exclude_from_sim no)
 		(in_bom yes)
@@
 		)
 		(property "Sheetfile" "target.kicad_sch"
-			(at 152.4 76.7846 0)
+			(at 152.4 79.3246 0)
 			(effects
 				(font
@@
 		)
 		(pin "RTS" input
-			(at 152.4 73.66 180)
+			(at 152.4 76.2 180)
 			(effects
 				(font
@@
 		)
 		(pin "RXD" output
-			(at 152.4 68.58 180)
+			(at 152.4 71.12 180)
 			(effects
 				(font
@@
 		)
 		(pin "TXD" input
-			(at 152.4 66.04 180)
+			(at 152.4 68.58 180)
 			(effects
 				(font
@@
 		)
 		(pin "DTR" input
-			(at 152.4 71.12 180)
-			(effects
-				(font
-					(size 1.27 1.27)
-				)
-				(justify left)
-			)
-		)
-		(instances
-			(project "XLink-HW"
+			(at 152.4 73.66 180)
+			(effects
+				(font
+					(size 1.27 1.27)
+				)
+				(justify left)
+			)
+		)
+		(pin "SWD_OEN" input
+			(at 152.4 63.5 180)
+			(effects
+				(font
+					(size 1.27 1.27)
+				)
+				(justify left)
+			)
+		)
+		(instances
+			(project "Aphid-HW"
 				(path "/023254f9-35e2-408c-9a7c-a91daeda5756"
 					(page "4")
@@
 	(sheet
 		(at 101.6 50.8)
-		(size 25.4 25.4)
+		(size 25.4 27.94)
 		(exclude_from_sim no)
 		(in_bom yes)
@@
 		)
 		(property "Sheetfile" "ftdi.kicad_sch"
-			(at 101.6 76.7846 0)
+			(at 101.6 79.3246 0)
 			(effects
 				(font
@@
 		)
 		(pin "DTR" output
+			(at 127 73.66 0)
+			(effects
+				(font
+					(size 1.27 1.27)
+				)
+				(justify right)
+			)
+		)
+		(pin "RTS" output
+			(at 127 76.2 0)
+			(effects
+				(font
+					(size 1.27 1.27)
+				)
+				(justify right)
+			)
+		)
+		(pin "RXD" input
 			(at 127 71.12 0)
-			(effects
-				(font
-					(size 1.27 1.27)
-				)
-				(justify right)
-			)
-		)
-		(pin "RTS" output
-			(at 127 73.66 0)
-			(effects
-				(font
-					(size 1.27 1.27)
-				)
-				(justify right)
-			)
-		)
-		(pin "RXD" input
-			(at 127 68.58 0)
 			(effects
 				(font
@@
 		)
 		(pin "TXD" output
-			(at 127 66.04 0)
-			(effects
-				(font
-					(size 1.27 1.27)
-				)
-				(justify right)
-			)
-		)
-		(instances
-			(project "XLink-HW"
+			(at 127 68.58 0)
+			(effects
+				(font
+					(size 1.27 1.27)
+				)
+				(justify right)
+			)
+		)
+		(pin "SWD_OEN" output
+			(at 127 63.5 0)
+			(effects
+				(font
+					(size 1.27 1.27)
+				)
+				(justify right)
+			)
+		)
+		(instances
+			(project "Aphid-HW"
 				(path "/023254f9-35e2-408c-9a7c-a91daeda5756"
 					(page "3")
@@
 		)
 		(instances
-			(project "XLink-HW"
+			(project "Aphid-HW"
 				(path "/023254f9-35e2-408c-9a7c-a91daeda5756"
 					(page "2")
