File: ftdi.kicad_sch (KiCad schematic)
At the start: 26 parts, among them U3 93LC56BT-I/OT, U4 FT2232HQ, Y1 ECS-120-20-33-CKM-TR

Commit message: Rework logic gates
Rename to aphid
Connections:
- net SWD_OEN: now reaches U4.26 (ACBUS0)
- no-connect marks 26 -> 25
Other:
- title: X-Link -> Aphid
Changed lines of the file:
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@@
 	(paper "A4")
 	(title_block
-		(title "X-Link")
-		(date "2026-02-28")
-		(rev "v1.0")
+		(title "Aphid")
+		(date "2026-03-21")
+		(rev "v1.1")
 		(company "TL Embedded")
 	)
@@
 	)
 	(no_connect
-		(at 204.47 80.01)
-	)
-	(no_connect
 		(at 204.47 92.71)
 	)
@@
 	(wire
 		(pts
+			(xy 204.47 80.01) (xy 215.9 80.01)
+		)
+		(stroke
+			(width 0)
+			(type default)
+		)
+	)
+	(wire
+		(pts
 			(xy 69.85 116.84) (xy 74.93 116.84)
 		)
@@
 		)
 	)
+	(hierarchical_label "SWD_OEN"
+		(shape output)
+		(at 215.9 80.01 0)
+		(effects
+			(font
+				(size 1.27 1.27)
+			)
+			(justify left)
+		)
+	)
 	(hierarchical_label "TDI"
 		(shape output)
@@
 	)
 	(symbol
+		(lib_name "+1V8_2")
 		(lib_id "power:+1V8")
 		(at 24.13 52.07 0)
@@
 	)
 	(symbol
+		(lib_name "+1V8_1")
 		(lib_id "power:+1V8")
 		(at 24.13 27.94 0)
@@
 	)
 	(symbol
+		(lib_name "GND_1")
 		(lib_id "power:GND")
 		(at 24.13 38.1 0)
@@
 	)
 	(symbol
+		(lib_name "GND_2")
 		(lib_id "power:GND")
 		(at 24.13 62.23 0)
