File: usb.kicad_sch (KiCad schematic)
At the start: 7 parts, among them J1 USB4105-GF-A-060, U1 USBLC6-2SC6, U2 MCP1755T-3302E/OT

Commit message: Rework logic gates
Rename to aphid
Other:
- title: X-Link -> Aphid
Changed lines of the file:
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@@
 	(paper "A4")
 	(title_block
-		(title "X-Link")
-		(date "2026-02-28")
-		(rev "v1.0")
+		(title "Aphid")
+		(date "2026-03-21")
+		(rev "v1.1")
 		(company "TL Embedded")
 	)
@@
 	)
 	(symbol
+		(lib_name "VBUS_1")
 		(lib_id "power:VBUS")
 		(at 93.98 52.07 0)
